File: kicad_files/Smart_Bed_Lamp.kicad_sch (KiCad schematic)
At the start: 0 parts

Commit message: Add files via upload
Other:
- note removed: "Barrel Jack"
- note removed: "LED"
- note removed: "USB-C"
