File: kicad_files/schematic.kicad_sch (KiCad schematic)
At the start: 54 parts, among them J1 USB_C_Receptacle_USB2.0_14P, J2 Barrel_Jack, Q1 MMBT3904, SW1 SW_Push, SW2 RST, SW3 BOOT, U1 ESP32-C3-WROOM-02, U2 TPS5430DDA, U3 AMS1117-3.3

Commit message: Add files via upload
Parts:
- added C9: 100nF, symbol Device:C_Small
- added J10, J11, J12: 5V, symbol Connector:Conn_01x01_Pin
- added J13: BOOT, symbol Connector:Conn_01x01_Pin
- added J14: RX/TX, symbol Connector:Conn_01x02_Pin
- added J15: IO0, symbol Connector:Conn_01x01_Pin
- added J16: IO1, symbol Connector:Conn_01x01_Pin
- added J17: IO3, symbol Connector:Conn_01x01_Pin
- added J18: IO4, symbol Connector:Conn_01x01_Pin
- added J3: IO7, symbol Connector:Conn_01x01_Pin
- added J4, J5, J6: 3V3, symbol Connector:Conn_01x01_Pin
- added J7, J8, J9: GND, symbol Connector:Conn_01x01_Pin
- added R9: 10K, symbol Device:R_Small
Connections:
- net 3V3: now also J4.1 (Pin_1), J5.1 (Pin_1), J6.1 (Pin_1), R9.1
- net 5V: now also J10.1 (Pin_1), J11.1 (Pin_1), J12.1 (Pin_1)
- net GND: now also SW1.1, C9.2, J7.1 (Pin_1), J8.1 (Pin_1), J9.1 (Pin_1)
- net at U1.11 (IO20/RXD): now also J14.2 (Pin_2)
- net at U1.12 (IO21/TXD): now also J14.1 (Pin_1)
- net IO3: now reaches U1.15 (IO3)
- net IO3: now also J17.1 (Pin_1)
- net IO1: now reaches U1.17 (IO1)
- net IO1: now also J16.1 (Pin_1)
- net IO0: now reaches U1.18 (IO0)
- net IO0: now also J15.1 (Pin_1)
- net IO4: now reaches U1.3 (IO4)
- net IO4: now also J18.1 (Pin_1)
- net at U1.6 (IO7): now also SW1.2, C9.1, J3.1 (Pin_1), R9.2
- net at JP2.1 (A), R7.2, SW3.2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: now also J13.1 (Pin_1)
- no-connect marks 4 -> 5
Other:
- note added: "Breakout pins"
- note added: "Buzzer"
- note added: "Connectors"
- note added: "Leds"
- note added: "MCU"
- moved on the sheet: BZ1, C1, C2, C3, C4, C5, C6, C7, C8, D1, D10, D11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

Commit message: Add files via upload
Parts:
- removed J14: RX/TX, symbol Connector:Conn_01x02_Pin
- added C10, C11, C12, C13, C14, C15, C16, C17, C18, C19, C20, C21, C22, C23, C24, C25, C26, C27, C28, C29: 100nF, Capacitor_SMD:C_0603_1608Metric, symbol Device:C_Small
- added J14: RX, TestPoint:TestPoint_THTPad_D2.0mm_Drill1.0mm, symbol Connector:Conn_01x01_Pin
- added J19: TX, TestPoint:TestPoint_THTPad_D2.0mm_Drill1.0mm, symbol Connector:Conn_01x01_Pin
- BZ1: footprint (none) -> Buzzer_Beeper:Buzzer_12x9.5RM7.6
- C1, C2, C3, C7, C8, C9: footprint (none) -> Capacitor_SMD:C_0603_1608Metric
- C4: footprint (none) -> Capacitor_THT:CP_Radial_D6.3mm_P2.50mm
- C5: footprint (none) -> Capacitor_THT:CP_Radial_D8.0mm_P3.50mm
- C6: footprint (none) -> Capacitor_SMD:C_0805_2012Metric
- J1: footprint (none) -> Connector_USB:USB_C_Receptacle_G-Switch_GT-USB-7010ASV
- J10, J11, J12, J13, J15, J16, J17, J18, J3, J4, J5, J6, J7, J8, J9: footprint (none) -> TestPoint:TestPoint_THTPad_D2.0mm_Drill1.0mm
- J2: footprint (none) -> Connector_BarrelJack:BarrelJack_CLIFF_FC681465S_SMT_Horizontal
- L1: footprint (none) -> Inductor_SMD:L_10.4x10.4_H4.8
- R1, R2, R3, R4, R5, R6, R7, R8, R9: footprint (none) -> Resistor_SMD:R_0603_1608Metric
- SW1, SW2, SW3: footprint (none) -> Button_Switch_THT:SW_PUSH_6mm
Connections:
- net 5V: now also C10.1, C11.1, C12.1, C13.1, C14.1, C15.1, C16.1, C17.1, C18.1, C19.1, C21.1, C22.1, C23.1, C24.1, C25.1, C26.1, C27.1, C28.1, C29.1
- net GND: now also C10.2, C11.2, C12.2, C13.2, C14.2, C15.2, C16.2, C17.2, C18.2, C19.2, C20.2, C21.2, C22.2, C23.2, C24.2, C25.2, C26.2, C27.2, C28.2, C29.2
- net at D1.1 (VDD), D21.1 (K): now also C20.1
- net at U1.11 (IO20/RXD): now also J14.1 (Pin_1)
- net at U1.12 (IO21/TXD): now also J19.1 (Pin_1)
